File: Thermography_EAGLE_FILES_COPY/wiring_thermography.brd (EAGLE design)
At the start: 71.1 x 64.4 mm, 19 parts

Commit message: updated eagle files
Parts:
- C(RCANALOGOUT): value (none) -> 10µ
- C(RCSWITCH): value (none) -> 10p
- R(ANALOGOUT): value (none) -> 160
- R1(RCSWITCH): value (none) -> 10
- R2(RCSWITCH): value (none) -> 16k
Changed lines of the file:
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@@
 <attribute name="VALUE" x="104.14" y="62.865" size="1.27" layer="27"/>
 </element>
-<element name="C(RCANALOGOUT)" library="capacitor-wima" library_urn="urn:adsk.eagle:library:116" package="C5B5" package3d_urn="urn:adsk.eagle:package:5428/1" value="" x="105.41" y="45.72" smashed="yes" rot="R90">
+<element name="C(RCANALOGOUT)" library="capacitor-wima" library_urn="urn:adsk.eagle:library:116" package="C5B5" package3d_urn="urn:adsk.eagle:package:5428/1" value="10µ" x="105.41" y="45.72" smashed="yes" rot="R90">
 <attribute name="NAME" x="102.616" y="43.18" size="1.27" layer="25" ratio="10" rot="R90"/>
 <attribute name="VALUE" x="107.696" y="43.18" size="1.27" layer="27" ratio="10" rot="R90"/>
 </element>
-<element name="C(RCSWITCH)" library="capacitor-wima" library_urn="urn:adsk.eagle:library:116" package="C5B5" package3d_urn="urn:adsk.eagle:package:5428/1" value="" x="43.18" y="39.37" smashed="yes" rot="R90">
+<element name="C(RCSWITCH)" library="capacitor-wima" library_urn="urn:adsk.eagle:library:116" package="C5B5" package3d_urn="urn:adsk.eagle:package:5428/1" value="10p" x="43.18" y="39.37" smashed="yes" rot="R90">
 <attribute name="NAME" x="40.386" y="36.83" size="1.27" layer="25" ratio="10" rot="R90"/>
 <attribute name="VALUE" x="45.466" y="36.83" size="1.27" layer="27" ratio="10" rot="R90"/>
@@
 <attribute name="VALUE" x="53.96" y="27.94" size="1.27" layer="27" rot="R180"/>
 </element>
-<element name="R1(RCSWITCH)" library="rcl" library_urn="urn:adsk.eagle:library:334" package="0207/7" package3d_urn="urn:adsk.eagle:package:23493/2" value="" x="43.18" y="62.23" smashed="yes" rot="R270">
+<element name="R1(RCSWITCH)" library="rcl" library_urn="urn:adsk.eagle:library:334" package="0207/7" package3d_urn="urn:adsk.eagle:package:23493/2" value="10" x="43.18" y="62.23" smashed="yes" rot="R270">
 <attribute name="NAME" x="44.577" y="64.77" size="1.27" layer="25" ratio="10" rot="R270"/>
 <attribute name="SPICEPREFIX" value="R" x="43.18" y="62.23" size="1.778" layer="27" rot="R270" display="off"/>
 <attribute name="VALUE" x="42.6212" y="64.516" size="1.27" layer="27" ratio="10" rot="R270"/>
 </element>
-<element name="R2(RCSWITCH)" library="rcl" library_urn="urn:adsk.eagle:library:334" package="0207/7" package3d_urn="urn:adsk.eagle:package:23493/2" value="" x="43.18" y="50.8" smashed="yes" rot="R270">
+<element name="R2(RCSWITCH)" library="rcl" library_urn="urn:adsk.eagle:library:334" package="0207/7" package3d_urn="urn:adsk.eagle:package:23493/2" value="16k" x="43.18" y="50.8" smashed="yes" rot="R270">
 <attribute name="NAME" x="44.577" y="53.34" size="1.27" layer="25" ratio="10" rot="R270"/>
 <attribute name="SPICEPREFIX" value="R" x="43.18" y="50.8" size="1.778" layer="27" rot="R270" display="off"/>
 <attribute name="VALUE" x="42.6212" y="53.086" size="1.27" layer="27" ratio="10" rot="R270"/>
 </element>
-<element name="R(ANALOGOUT)" library="rcl" library_urn="urn:adsk.eagle:library:334" package="0207/7" package3d_urn="urn:adsk.eagle:package:23493/2" value="" x="105.41" y="57.15" smashed="yes" rot="R270">
+<element name="R(ANALOGOUT)" library="rcl" library_urn="urn:adsk.eagle:library:334" package="0207/7" package3d_urn="urn:adsk.eagle:package:23493/2" value="160" x="105.41" y="57.15" smashed="yes" rot="R270">
 <attribute name="NAME" x="106.807" y="59.69" size="1.27" layer="25" ratio="10" rot="R270"/>
 <attribute name="SPICEPREFIX" value="R" x="105.41" y="57.15" size="1.778" layer="27" rot="R270" display="off"/>
